File: PCB/1.2/schTop.kicad_sch (KiCad schematic)
At the start: 88 parts, among them J1 USB-Micro, J2 TSM-108-01-T-SH-A-P-TR, J3 Raspberry-Pi_2x5-Pin_Header, J4 Conn_02x03_Odd_Even, J5 USB_C_Receptacle, Q1 BSS84AK,215, Q2 BSS84AK,215, Q3 BSS84AK,215, Q4 Q_NMOS_GSD, U1 CP2102N-A02-GQFN24R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

Commit message: Updating the PCB to remove the test points from the BOM and also to substitute the raspberry pi header part number because the previous one was out of stock in JLCPCB.
Parts:
- J2: footprint Connector_8-pin_SMT_hole_1.5mm -> rs485RPihat:Connector_8-pin_SMT_hole_1.5mm
- J3: Alternative Part Number (none) -> C261072; LCSC C261072 -> C843271; PartNumber C261072 -> (none)
- TP15, TP16, TP17, TP18, TP19, TP20, TP21, TP22, TP23: now left out of the parts list
Changed lines of the file:
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@@
 			)
 		)
-		(property "PartNumber" "C261072"
+		(property "Digikey" "_"
 			(at 133.985 174.625 0)
 			(effects
@@
 			)
 		)
-		(property "Digikey" "_"
+		(property "LCSC" "C843271 "
 			(at 133.985 174.625 0)
 			(effects
@@
 			)
 		)
-		(property "LCSC" "C261072"
+		(property "Alternative Part Number" "C261072"
 			(at 133.985 174.625 0)
 			(effects
 				(font
-					(size 0.889 0.889)
+					(size 1.27 1.27)
 				)
 				(hide yes)
@@
 			)
 		)
-		(property "Footprint" "Connector_8-pin_SMT_hole_1.5mm"
+		(property "Footprint" "rs485RPihat:Connector_8-pin_SMT_hole_1.5mm"
 			(at 153.67 97.79 0)
 			(effects
@@
 		(unit 1)
 		(exclude_from_sim no)
-		(in_bom yes)
+		(in_bom no)
 		(on_board yes)
 		(dnp no)
@@
 		(unit 1)
 		(exclude_from_sim no)
-		(in_bom yes)
+		(in_bom no)
 		(on_board yes)
 		(dnp no)
@@
 		(unit 1)
 		(exclude_from_sim no)
-		(in_bom yes)
+		(in_bom no)
 		(on_board yes)
 		(dnp no)
@@
 		(unit 1)
 		(exclude_from_sim no)
-		(in_bom yes)
+		(in_bom no)
 		(on_board yes)
 		(dnp no)
@@
 		(unit 1)
 		(exclude_from_sim no)
-		(in_bom yes)
+		(in_bom no)
 		(on_board yes)
 		(dnp no)
@@
 		(unit 1)
 		(exclude_from_sim no)
-		(in_bom yes)
+		(in_bom no)
 		(on_board yes)
 		(dnp no)
@@
 		(unit 1)
 		(exclude_from_sim no)
-		(in_bom yes)
+		(in_bom no)
 		(on_board yes)
 		(dnp no)
@@
 		(unit 1)
 		(exclude_from_sim no)
-		(in_bom yes)
+		(in_bom no)
 		(on_board yes)
 		(dnp no)
@@
 		(unit 1)
 		(exclude_from_sim no)
-		(in_bom yes)
+		(in_bom no)
 		(on_board yes)
 		(dnp no)
